File: eagle/v0.2.brd (EAGLE design)
At the start: 85 x 90 mm, 3 parts

Commit message: More work on the PCB.
Parts:
- added 100NF, 10UF: (no value), rcl:C025-025X050
- added MCP4921: (no value), ic-package:DIL08
- moved RPI 6.40 mm to (35.0, 45.0)
Connections:
- new net 5V: 100NF.1, 10UF.1, MCP4921.1, RPI.2
- new net SPIO_CS1: MCP4921.2, RPI.26
- net 3.3V: now also MCP4921.6
- net GND: now also 100NF.2, 10UF.2, MCP4921.5, MCP4921.7
- net SPI0_CS0: now also MCP4921.4
- net SPI0_SCK: now also MCP4921.3
Routing:
- net 5V: track 0.00 -> 88.2 mm
- net SPI0_SCK: track 29.3 -> 76.7 mm
- net 3.3V: track 68.6 -> 113.0 mm
- net GND: track 72.7 -> 113.6 mm
- net SPI0_CS0: track 42.6 -> 81.8 mm
- net SPIO_CS1: track 0.00 -> 36.3 mm
- net SPI1_CS: track 59.5 -> 74.1 mm
- net SPI1_MISO: track 21.5 -> 28.0 mm
- net SPI1_SCK: track 24.1 -> 30.5 mm
- net SPI1_MOSI: track 24.0 -> 30.5 mm
- net SPI1_RST: track 22.1 -> 27.4 mm
- net SPI0_RESET: track 37.5 -> 40.3 mm
- net SPI0_MISO: track 24.7 -> 27.5 mm
- net SPI0_DC_RS: track 29.3 -> 32.1 mm
- net SPI0_LED: track 25.2 -> 27.9 mm
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Other:
- board size 85 x 90 mm -> 85 x 95 mm
- board text added: "2.2" SPI LCD"
- board text added: "SPI RFID"
