File: eagle/v0.2.sch (EAGLE design)
At the start: 3 parts

Commit message: More work on the PCB.
Parts:
- added 100NF, 10UF: (no value), rcl:C-EU025-025X050
- added MCP4921: (no value), ic-package:DIL8
Connections:
- new net 5V: 100NF.1, 10UF.1, MCP4921.1, RPI-2.KL
- new net SPIO_CS1: MCP4921.2, RPI-26.KL
- net 3.3V: now also MCP4921.6
- net GND: now also 100NF.2, 10UF.2, MCP4921.5, MCP4921.7
- net SPI0_CS0: now also MCP4921.4
- net SPI0_SCK: now also MCP4921.3
Other:
- moved on the sheet: LCD, RFID
