File: eagle/v0.3.brd (EAGLE design)
At the start: 96 x 95 mm, 10 parts

Commit message: Correct lipo connections.
Connections:
- removed net N$1: LIPO.3, RPI.3
- removed net N$14: LIPO.14, RPI.14
- removed net N$2: LIPO.4, RPI.4
- removed net N$3: LIPO.5, RPI.5
- removed net N$5: LIPO.8, RPI.8
- removed net N$6: LIPO.9, RPI.9
- removed net N$7: LIPO.10, RPI.10
- removed net N$8: LIPO.11, RPI.11
- removed net N$9: LIPO.13, RPI.13
- net SPI1_CS: no longer LIPO.12
Routing:
- net N$9: track 61.0 -> 0.00 mm
- net N$14: track 58.0 -> 0.00 mm
- net N$5: track 57.2 -> 0.00 mm
- net N$7: track 57.1 -> 0.00 mm
- net N$2: track 57.1 -> 0.00 mm
- net N$8: track 57.1 -> 0.00 mm
- net N$3: track 57.1 -> 0.00 mm
- net N$1: track 57.1 -> 0.00 mm
- net N$6: track 57.1 -> 0.00 mm
Changed lines of the file:
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@@
 <contactref element="RPI" pad="12"/>
 <contactref element="RFID" pad="8"/>
-<contactref element="LIPO" pad="12"/>
 <wire x1="81.3816" y1="56.5404" x2="37.338" y2="56.5404" width="0.1524" layer="16"/>
 <wire x1="37.338" y1="56.5404" x2="36.2712" y2="56.5404" width="0.1524" layer="16"/>
@@
 <wire x1="90.2208" y1="63.8556" x2="89.154" y2="62.7888" width="0.1524" layer="16"/>
 <wire x1="36.2712" y1="56.5404" x2="36.27" y2="56.43" width="0.1524" layer="16"/>
-<wire x1="90.2208" y1="63.8556" x2="90.27" y2="63.92" width="0.1524" layer="16"/>
 <wire x1="10.0584" y1="8.0772" x2="10.0584" y2="7.7724" width="0.1524" layer="1"/>
 <wire x1="8.382" y1="9.7536" x2="10.0584" y2="8.0772" width="0.1524" layer="1"/>
@@
 <wire x1="87.63" y1="68.8848" x2="87.73" y2="69" width="0.1524" layer="1"/>
 </signal>
-<signal name="N$14">
-<contactref element="LIPO" pad="14"/>
-<contactref element="RPI" pad="14"/>
-<wire x1="78.7908" y1="53.9496" x2="36.2712" y2="53.9496" width="0.1524" layer="1"/>
-<wire x1="87.3252" y1="62.484" x2="78.7908" y2="53.9496" width="0.1524" layer="1"/>
-<wire x1="89.154" y1="62.484" x2="87.3252" y2="62.484" width="0.1524" layer="1"/>
-<wire x1="90.2208" y1="61.4172" x2="89.154" y2="62.484" width="0.1524" layer="1"/>
-<wire x1="36.2712" y1="53.9496" x2="36.27" y2="53.89" width="0.1524" layer="1"/>
-<wire x1="90.2208" y1="61.4172" x2="90.27" y2="61.38" width="0.1524" layer="1"/>
-</signal>
-<signal name="N$1">
-<contactref element="LIPO" pad="3"/>
-<contactref element="RPI" pad="3"/>
-<wire x1="34.7472" y1="66.5988" x2="33.8328" y2="66.5988" width="0.1524" layer="16"/>
-<wire x1="36.2712" y1="68.1228" x2="34.7472" y2="66.5988" width="0.1524" layer="16"/>
-<wire x1="81.6864" y1="68.1228" x2="36.2712" y2="68.1228" width="0.1524" layer="16"/>
-<wire x1="87.63" y1="74.0664" x2="81.6864" y2="68.1228" width="0.1524" layer="16"/>
-<wire x1="33.8328" y1="66.5988" x2="33.73" y2="66.59" width="0.1524" layer="16"/>
-<wire x1="87.63" y1="74.0664" x2="87.73" y2="74.08" width="0.1524" layer="16"/>
-</signal>
-<signal name="N$2">
-<contactref element="RPI" pad="4"/>
-<contactref element="LIPO" pad="4"/>
-<wire x1="81.3816" y1="66.5988" x2="36.2712" y2="66.5988" width="0.1524" layer="1"/>
-<wire x1="87.7824" y1="72.9996" x2="81.3816" y2="66.5988" width="0.1524" layer="1"/>
-<wire x1="89.154" y1="72.9996" x2="87.7824" y2="72.9996" width="0.1524" layer="1"/>
-<wire x1="90.2208" y1="74.0664" x2="89.154" y2="72.9996" width="0.1524" layer="1"/>
-<wire x1="36.2712" y1="66.5988" x2="36.27" y2="66.59" width="0.1524" layer="1"/>
-<wire x1="90.2208" y1="74.0664" x2="90.27" y2="74.08" width="0.1524" layer="1"/>
-</signal>
-<signal name="N$3">
-<contactref element="LIPO" pad="5"/>
-<contactref element="RPI" pad="5"/>
-<wire x1="34.8996" y1="64.1604" x2="33.8328" y2="64.1604" width="0.1524" layer="1"/>
-<wire x1="36.2712" y1="65.532" x2="34.8996" y2="64.1604" width="0.1524" layer="1"/>
-<wire x1="81.6864" y1="65.532" x2="36.2712" y2="65.532" width="0.1524" layer="1"/>
-<wire x1="87.63" y1="71.4756" x2="81.6864" y2="65.532" width="0.1524" layer="1"/>
-<wire x1="33.8328" y1="64.1604" x2="33.73" y2="64.05" width="0.1524" layer="1"/>
-<wire x1="87.63" y1="71.4756" x2="87.73" y2="71.54" width="0.1524" layer="1"/>
-</signal>
 <signal name="N$4">
 <contactref element="RPI" pad="6"/>
@@
 <wire x1="90.2208" y1="71.4756" x2="90.27" y2="71.54" width="0.1524" layer="1"/>
 </signal>
-<signal name="N$5">
-<contactref element="LIPO" pad="8"/>
-<contactref element="RPI" pad="8"/>
-<wire x1="81.3816" y1="61.5696" x2="36.2712" y2="61.5696" width="0.1524" layer="1"/>
-<wire x1="87.7824" y1="67.9704" x2="81.3816" y2="61.5696" width="0.1524" layer="1"/>
-<wire x1="89.3064" y1="67.9704" x2="87.7824" y2="67.9704" width="0.1524" layer="1"/>
-<wire x1="90.2208" y1="68.8848" x2="89.3064" y2="67.9704" width="0.1524" layer="1"/>
-<wire x1="36.2712" y1="61.5696" x2="36.27" y2="61.51" width="0.1524" layer="1"/>
-<wire x1="90.2208" y1="68.8848" x2="90.27" y2="69" width="0.1524" layer="1"/>
-</signal>
-<signal name="N$6">
-<contactref element="RPI" pad="9"/>
-<contactref element="LIPO" pad="9"/>
-<wire x1="34.7472" y1="58.9788" x2="33.8328" y2="58.9788" width="0.1524" layer="1"/>
-<wire x1="36.2712" y1="60.5028" x2="34.7472" y2="58.9788" width="0.1524" layer="1"/>
-<wire x1="81.6864" y1="60.5028" x2="36.2712" y2="60.5028" width="0.1524" layer="1"/>
-<wire x1="87.63" y1="66.4464" x2="81.6864" y2="60.5028" width="0.1524" layer="1"/>
-<wire x1="33.8328" y1="58.9788" x2="33.73" y2="58.97" width="0.1524" layer="1"/>
-<wire x1="87.63" y1="66.4464" x2="87.73" y2="66.46" width="0.1524" layer="1"/>
-</signal>
-<signal name="N$7">
-<contactref element="LIPO" pad="10"/>
-<contactref element="RPI" pad="10"/>
-<wire x1="81.3816" y1="58.9788" x2="36.2712" y2="58.9788" width="0.1524" layer="1"/>
-<wire x1="87.7824" y1="65.3796" x2="81.3816" y2="58.9788" width="0.1524" layer="1"/>
-<wire x1="89.154" y1="65.3796" x2="87.7824" y2="65.3796" width="0.1524" layer="1"/>
-<wire x1="90.2208" y1="66.4464" x2="89.154" y2="65.3796" width="0.1524" layer="1"/>
-<wire x1="36.2712" y1="58.9788" x2="36.27" y2="58.97" width="0.1524" layer="1"/>
-<wire x1="90.2208" y1="66.4464" x2="90.27" y2="66.46" width="0.1524" layer="1"/>
-</signal>
-<signal name="N$8">
-<contactref element="RPI" pad="11"/>
-<contactref element="LIPO" pad="11"/>
-<wire x1="34.8996" y1="56.5404" x2="33.8328" y2="56.5404" width="0.1524" layer="1"/>
-<wire x1="36.2712" y1="57.912" x2="34.8996" y2="56.5404" width="0.1524" layer="1"/>
-<wire x1="81.6864" y1="57.912" x2="36.2712" y2="57.912" width="0.1524" layer="1"/>
-<wire x1="87.63" y1="63.8556" x2="81.6864" y2="57.912" width="0.1524" layer="1"/>
-<wire x1="33.8328" y1="56.5404" x2="33.73" y2="56.43" width="0.1524" layer="1"/>
-<wire x1="87.63" y1="63.8556" x2="87.73" y2="63.92" width="0.1524" layer="1"/>
-</signal>
-<signal name="N$9">
-<contactref element="RPI" pad="13"/>
-<contactref element="LIPO" pad="13"/>
-<wire x1="33.8328" y1="52.7304" x2="33.8328" y2="53.7972" width="0.1524" layer="1"/>
-<wire x1="35.2044" y1="51.3588" x2="33.8328" y2="52.7304" width="0.1524" layer="1"/>
-<wire x1="35.2044" y1="50.9016" x2="35.2044" y2="51.3588" width="0.1524" layer="1"/>
-<wire x1="35.814" y1="50.292" x2="35.2044" y2="50.9016" width="0.1524" layer="1"/>
-<wire x1="76.6572" y1="50.292" x2="35.814" y2="50.292" width="0.1524" layer="1"/>
-<wire x1="87.63" y1="61.2648" x2="76.6572" y2="50.292" width="0.1524" layer="1"/>
-<wire x1="33.8328" y1="53.7972" x2="33.73" y2="53.89" width="0.1524" layer="1"/>
-<wire x1="87.63" y1="61.2648" x2="87.73" y2="61.38" width="0.1524" layer="1"/>
-</signal>
 <signal name="N$10">
