File: eagle/v0.6.brd (EAGLE design)
At the start: 96 x 95 mm, 15 parts, among them IC1 LM386N-1

Commit message: Let's do another run of boards, this time with more LEDs and sound half done.
Parts:
- removed 0.1UF: (no value), rcl:C025-025X050
- removed 10OHM, RLED: (no value), rcl:0204/5
- removed IC1: LM386N-1, linear:DIL08
- removed U$1: XD-2308-01-R, XD-2308-01-R speaker:XD-2308-01-R
- added 150OHM1, 270OHM1, RLED1, RLED2, RLED3: (no value), rcl:0204/5
- added 33NF1: (no value), rcl:C025-025X050
- added AUDIOOUT: (no value), con-lstb:MA03-1
- added LED2, LED3: (no value), led:LED3MM
- moved LED1 14.1 mm to (85.0, 14.0)
- moved 10UF 8.00 mm to (91.0, 38.0)
- moved 150OHM 8.00 mm to (83.0, 38.0)
- moved 270OHM 8.00 mm to (83.0, 44.0)
- moved 33NF 8.00 mm to (91.0, 44.0)
- renumbered 1000UF to 10UF1
Connections:
- net AUDIO renamed AUDIO1
- new net AUDIO2: 270OHM1.2, RPI.18
- new net N$3: LED3.A, RLED3.2
- new net N$4: RLED1.1, RPI.29
- new net N$9: 10UF1.1, AUDIOOUT.3
- net 5V: no longer IC1.6
- net GND: now also 150OHM1.1, 33NF1.1, AUDIOOUT.2, LED2.K, LED3.K; no longer 10OHM.1, IC1.2, IC1.4, U$1.-
- net N$1: now also 150OHM.2
- net N$11: now also RLED1.2; no longer RLED.2
- net N$2: now also LED2.A, RLED2.2; no longer 10UF.1, 150OHM.2, IC1.3
- net N$5: now also RLED2.1, RPI.31; no longer RLED.1, RPI.18
- net N$6: now also RLED3.1, RPI.32; no longer 0.1UF.2, 10UF1.2, IC1.5
- net N$7: now also 10UF1.2, 150OHM1.2, 270OHM1.1, 33NF1.2; no longer 10UF1.1, U$1.+
- net N$8: now also 10UF.1, AUDIOOUT.1; no longer 0.1UF.1, 10OHM.2
Routing:
- net AUDIO2: track 0.00 -> 53.7 mm
- net N$4: track 0.00 -> 48.9 mm
- net 5V: track 101.8 -> 58.9 mm
- net AUDIO1: track 48.5 -> 76.6 mm, vias 0 -> 2
- net N$6: track 22.7 -> 50.3 mm
- net N$9: track 0.00 -> 14.4 mm
- net N$2: track 17.2 -> 4.23 mm
- net N$5: track 51.0 -> 61.7 mm
- net GND: track 276.4 -> 266.0 mm, vias 0 -> 1
- net N$7: track 23.9 -> 14.7 mm
- net N$1: track 11.4 -> 17.6 mm
- net N$8: track 11.7 -> 6.76 mm
- net N$3: track 0.00 -> 4.36 mm
- net LCD_RESET: track 44.0 -> 42.3 mm
- net N$11: track 5.97 -> 4.38 mm
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Other:
- board text added: "GangScan v0.6"
- board text removed: "GangScan v0.5"
