File: eagle/v0.6.sch (EAGLE design)
At the start: 15 parts, among them IC1 LM386N-1

Commit message: Let's do another run of boards, this time with more LEDs and sound half done.
Parts:
- removed 0.1UF, 1000UF: (no value), rcl:C-EU025-025X050
- removed 10OHM, RLED: (no value), rcl:R-US_0204/5
- removed IC1: LM386N-1, linear:LM386N-1
- removed U$1: XD-2308-01-R, XD-2308-01-R speaker:XD-2308-01-R
- added 10UF1, 33NF1: (no value), rcl:C-EU025-025X050
- added 150OHM1, 270OHM1, RLED1, RLED2, RLED3: (no value), rcl:R-US_0204/5
- added AUDIOOUT: (no value), con-lstb:MA03-1
- added LED2, LED3: (no value), led:LED3MM
Connections:
- net AUDIO renamed AUDIO1
- new net AUDIO2: 270OHM1.2, RPI-18.KL
- new net N$3: LED3.A, RLED3.2
- new net N$4: RLED1.1, RPI-29.KL
- new net N$9: 10UF1.1, AUDIOOUT.3
- net 5V: no longer IC1.VS
- net GND: now also 150OHM1.1, 33NF1.1, AUDIOOUT.2, LED2.C, LED3.C; no longer 10OHM.1, IC1.-IN, IC1.GND, U$1.-
- net N$1: now also 150OHM.2
- net N$11: now also RLED1.2; no longer RLED.2
- net N$2: now also LED2.A, RLED2.2; no longer 10UF.1, 150OHM.2, IC1.+IN
- net N$5: now also RLED2.1, RPI-31.KL; no longer RLED.1, RPI-18.KL
- net N$6: now also RLED3.1, RPI-32.KL; no longer 0.1UF.2, 1000UF.2, IC1.OUT
- net N$7: now also 10UF1.2, 150OHM1.2, 270OHM1.1, 33NF1.2; no longer 1000UF.1, U$1.+
- net N$8: now also 10UF.1, AUDIOOUT.1; no longer 0.1UF.1, 10OHM.2
Other:
- moved on the sheet: 10UF, 150OHM, 270OHM, 33NF
