File: eagle/v0.7.brd (EAGLE design)
At the start: 96 x 95 mm, 19 parts

Commit message: Board version v0.7
Parts:
- removed 10UF, 33NF, 33NF1: (no value), rcl:C025-025X050
- added C1, C2: 33nF, capacitor-wima:C5B5
- added E1: 1uF, rcl:C025-025X050
- E2: value (none) -> 1uF
- moved AUDIOOUT 3.61 mm to (87.0, 35.0)
- moved 150OHM 3.00 mm to (83.0, 41.0)
- moved 270OHM1 3.00 mm to (83.0, 23.0)
- renumbered 10UF1 to E2
Connections:
- net GND: now also C1.1, C2.1; no longer 33NF.1, 33NF1.1
- net N$1: now also C1.2, E1.2; no longer 10UF.2, 33NF.2
- net N$7: now also C2.2; no longer 33NF1.2
- net N$8: now also E1.1; no longer 10UF.1
Routing:
- net GND: track 291.8 -> 278.9 mm
- net N$5: track 61.7 -> 50.3 mm
- net N$6: track 59.2 -> 50.3 mm
- net N$9: track 14.4 -> 18.3 mm
- net N$1: track 17.6 -> 14.1 mm
- net N$7: track 14.7 -> 12.3 mm
- net SPI0_CS1: track 50.8 -> 53.2 mm
- net AUDIO2: track 53.7 -> 54.9 mm
- net N$4: track 49.9 -> 48.9 mm
- net N$8: track 6.76 -> 6.13 mm
